File: PTnglieder.kicad_pcb (KiCad board)
At the start: 2 copper layers, 100 x 100 mm, 59 parts, among them J1 PT1, J2 PT2, J3 PT3, J4 GND, J5 USB_C_Receptacle_USB2.0, J6 PROG, J7 DEBUG, K1 G6K-2, Q1 BC847, SW1 LOAD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

Commit message: Update to new libs
Parts:
- moved D2 60.3 mm to (56.8, 79.9)
- moved R7 4.95 mm to (64.6, 82.7), turned to 180 degrees
- moved R2 1.54 mm to (68.5, 82.7)
- moved R1 1.31 mm to (72.3, 82.7)
- moved Q1 0.90 mm to (63.1, 79.9), turned to 180 degrees
- turned JP2 to 180 degrees
Routing:
- net Net-(D2-Pad2): track 6.32 -> 9.83 mm
- net -6V: track 80.9 -> 83.6 mm
- net Net-(Q1-Pad1): track 1.85 -> 4.39 mm
- net Net-(JP1-Pad2): track 25.0 -> 23.5 mm
- net Net-(R2-Pad2): track 2.57 -> 4.05 mm
- net Net-(K1-Pad7): track 15.3 -> 16.4 mm
- net Net-(C3-Pad1): track 52.4 -> 51.4 mm
- net SW: track 112.7 -> 112.1 mm
- net GND: vias 21 -> 32
Other:
- rule trace_min: 0.2 -> 0
- board text added: "1"
