File: PTnglieder.sch (KiCad schematic (older format))
At the start: 59 parts, among them J1 PT1, J2 PT2, J3 PT3, J4 GND, J5 USB_C_Receptacle_USB2.0, J6 PROG, J7 DEBUG, K1 G6K-2, Q1 BC847, SW1 LOAD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

Commit message: Update to new libs
Parts:
- J5: symbol Connector:USB_C_Receptacle_USB2.0 -> PTnglieder-rescue:USB_C_Receptacle_USB2.0-Connector
Changed lines of the file:
@@
 $EndComp
 $Comp
-L Connector:USB_C_Receptacle_USB2.0 J5
+L PTnglieder-rescue:USB_C_Receptacle_USB2.0-Connector J5
 U 1 1 5F77DF03
 P 1250 6700
